File: pcb/control/control.kicad_pcb (KiCad board)
At the start: 2 copper layers, 56 x 65.4 mm, 15 parts, among them J1 24v DC, J2 ESC Left, J3 ESC Right, J4 Buttons, J5 Joystick, J6 Lights, Q1 2N7002HSX, Q2 2N7002HSX, U1 L7805, U2 Pico

Commit message: Updated pcb
Parts:
- added G1: LOGO, OneTouch_Logo:onetouchlogo, F.Cu at (72.8, 104.8)
- added G2: LOGO, OneTouch_Logo:onetouchlogo, F.Cu at (132.5, 73.5)
- added H10: MountingHole, MountingHole:MountingHole_3.2mm_M3, F.Cu at (150.0, 69.0)
- added H11: MountingHole, MountingHole:MountingHole_3.2mm_M3, F.Cu at (122.0, 76.0)
- added H12: MountingHole, MountingHole:MountingHole_3.2mm_M3, F.Cu at (150.0, 111.0)
- added H13: MountingHole, MountingHole:MountingHole_3.2mm_M3, F.Cu at (122.0, 128.0)
- added H5: MountingHole, MountingHole:MountingHole_12.7mm, F.Cu at (137.0, 60.0)
- added H6: MountingHole, MountingHole:MountingHole_12.7mm, F.Cu at (137.0, 90.0)
- added H7: MountingHole, MountingHole:MountingHole_12.7mm, F.Cu at (137.0, 120.0)
- added H8: MountingHole, MountingHole:MountingHole_3.2mm_M3, F.Cu at (122.0, 104.0)
- added H9: MountingHole, MountingHole:MountingHole_3.2mm_M3, F.Cu at (122.0, 52.0)
- added J10: GND, Connector_Wire:SolderWire-0.75sqmm_1x01_D1.25mm_OD2.3mm, F.Cu at (130.0, 53.0)
- added J11: GND, Connector_Wire:SolderWire-0.75sqmm_1x01_D1.25mm_OD2.3mm, F.Cu at (130.0, 83.0)
- added J13: GND, Connector_Wire:SolderWire-0.75sqmm_1x01_D1.25mm_OD2.3mm, F.Cu at (130.0, 113.0)
- added J14: 1, Connector_Wire:SolderWire-0.75sqmm_1x01_D1.25mm_OD2.3mm, F.Cu at (130.0, 67.0)
- added J15: 2, Connector_Wire:SolderWire-0.75sqmm_1x01_D1.25mm_OD2.3mm, F.Cu at (130.0, 97.0)
- added J16: 3, Connector_Wire:SolderWire-0.75sqmm_1x01_D1.25mm_OD2.3mm, F.Cu at (130.0, 127.0)
- added J17: LED +, Connector_Wire:SolderWire-0.75sqmm_1x01_D1.25mm_OD2.3mm, F.Cu at (144.0, 67.0)
- added J18: LED +, Connector_Wire:SolderWire-0.75sqmm_1x01_D1.25mm_OD2.3mm, F.Cu at (144.0, 97.0)
- added J19: LED +, Connector_Wire:SolderWire-0.75sqmm_1x01_D1.25mm_OD2.3mm, F.Cu at (144.0, 127.0)
- added J20: LED -, Connector_Wire:SolderWire-0.75sqmm_1x01_D1.25mm_OD2.3mm, F.Cu at (144.0, 53.0)
- added J21: LED -, Connector_Wire:SolderWire-0.75sqmm_1x01_D1.25mm_OD2.3mm, F.Cu at (144.0, 83.0)
- added J22: LED -, Connector_Wire:SolderWire-0.75sqmm_1x01_D1.25mm_OD2.3mm, F.Cu at (144.0, 113.0)
- added J23: Joystick, Connector_Wire:SolderWire-0.75sqmm_1x05_P7mm_D1.25mm_OD3.5mm, F.Cu at (151.0, 104.0)
- added J24: Joystick, Connector_JST:JST_XH_B5B-XH-AM_1x05_P2.50mm_Vertical, F.Cu at (122.0, 69.0)
- added J25: Panel Lights, Connector_JST:JST_XH_B4B-XH-AM_1x04_P2.50mm_Vertical, F.Cu at (122.0, 94.0)
- added J26: Panel Buttons, Connector_JST:JST_XH_B4B-XH-AM_1x04_P2.50mm_Vertical, F.Cu at (122.0, 120.5)
- added J7: Panel Lights, Connector_JST:JST_XH_B4B-XH-AM_1x04_P2.50mm_Vertical, F.Cu at (110.5, 83.1)
- added T1: STD40NF10, STD40NF10:D_PAK, F.Cu at (82.8, 105.0)
- J4: value Buttons -> Panel Buttons
- J5: value Joystick -> Strip light; footprint Connector_JST:JST_XH_B5B-XH-AM_1x05_P2.50mm_Vertical -> Connector_JST:JST_XH_B2B-XH-A_1x02_P2.50mm_Vertical
- J6: value Lights -> Joystick; footprint Connector_JST:JST_XH_B4B-XH-AM_1x04_P2.50mm_Vertical -> Connector_JST:JST_XH_B5B-XH-AM_1x05_P2.50mm_Vertical
- moved J5 23.4 mm to (110.5, 92.2)
- moved J4 17.2 mm to (95.0, 104.4), turned to 0 degrees
- moved J6 13.9 mm to (110.5, 69.2)
Connections:
- J5 pad 1: GND -> Net-(J5-Pad1)
- J5 pad 2: Net-(J5-Pad2) -> +24V
- J6 pad 1: Net-(J6-Pad1) -> GND
- J6 pad 2: Net-(J6-Pad2) -> +3V3
- J6 pad 4: +24V -> Net-(J6-Pad4)
- Q1 pad 3: Net-(J6-Pad3) -> Net-(J7-Pad3)
- Q1 pad 6: Net-(J6-Pad2) -> Net-(J7-Pad2)
- Q2 pad 3: Net-(J6-Pad1) -> Net-(J7-Pad1)
- U2 pad 20: unconnected-(U2-Pad20) -> Net-(T1-Pad1)
- U2 pad 31: Net-(J5-Pad3) -> Net-(J6-Pad3)
- U2 pad 32: Net-(J5-Pad4) -> Net-(J6-Pad4)
- U2 pad 34: Net-(J5-Pad5) -> Net-(J6-Pad5)
- U2 pad 36: Net-(J5-Pad2) -> +3V3
Routing:
- net Net-(J19-Pad1): track 0.00 -> 109.1 mm
- net Net-(J12-Pad3): track 0.00 -> 56.3 mm
- net Net-(J14-Pad1): track 0.00 -> 51.9 mm
- net Net-(J8-Pad4): track 0.00 -> 48.7 mm
- net Net-(J8-Pad3): track 0.00 -> 43.1 mm
- net Net-(J8-Pad1): track 0.00 -> 41.0 mm
- net Net-(J5-Pad1): track 0.00 -> 39.8 mm
- net Net-(J8-Pad2): track 0.00 -> 39.0 mm
- net Net-(J12-Pad1): track 0.00 -> 33.2 mm
- net +24V: track 95.2 -> 127.1 mm
- net Net-(J5-Pad2): track 25.9 -> 0.00 mm
- net +3V3: track 0.00 -> 25.9 mm
- net Net-(J12-Pad2): track 0.00 -> 25.5 mm
- net Net-(J9-Pad2): track 0.00 -> 24.3 mm
- net Net-(J5-Pad3): track 16.2 -> 0.00 mm
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Other:
- board size 56 x 65.4 mm -> 95 x 88.5 mm
- board text added: "Donie Kelly © 2022"

Commit message: v2 of design
Parts:
- removed H11: MountingHole, MountingHole:MountingHole_3.2mm_M3
- removed J13: GND, Connector_Wire:SolderWire-0.75sqmm_1x01_D1.25mm_OD2.3mm
- removed J14: 1, Connector_Wire:SolderWire-0.75sqmm_1x01_D1.25mm_OD2.3mm
- removed J15: 2, Connector_Wire:SolderWire-0.75sqmm_1x01_D1.25mm_OD2.3mm
- removed J16: 3, Connector_Wire:SolderWire-0.75sqmm_1x01_D1.25mm_OD2.3mm
- removed J17, J18, J19: LED +, Connector_Wire:SolderWire-0.75sqmm_1x01_D1.25mm_OD2.3mm
- removed J20, J21, J22: LED -, Connector_Wire:SolderWire-0.75sqmm_1x01_D1.25mm_OD2.3mm
- removed J23: Joystick, Connector_Wire:SolderWire-0.75sqmm_1x05_P7mm_D1.25mm_OD3.5mm
- removed J24: Joystick, Connector_JST:JST_XH_B5B-XH-AM_1x05_P2.50mm_Vertical
- removed J25: Panel Lights, Connector_JST:JST_XH_B4B-XH-AM_1x04_P2.50mm_Vertical
- removed J26, J4: Panel Buttons, Connector_JST:JST_XH_B4B-XH-AM_1x04_P2.50mm_Vertical
- added J12: Switch 3, Connector_JST:JST_XH_B4B-XH-AM_1x04_P2.50mm_Vertical, F.Cu at (143.6, 126.0)
- added J8: Joystick, Connector_JST:JST_XH_B5B-XH-A_1x05_P2.50mm_Vertical, F.Cu at (150.6, 83.5)
- added J9: Cutout, Connector_JST:JST_XH_B2B-XH-AM_1x02_P2.50mm_Vertical, F.Cu at (121.6, 68.5)
- added R1: 1K, Resistor_SMD:R_1206_3216Metric, F.Cu at (138.5, 99.0)
- added R2: 15K, Resistor_SMD:R_1206_3216Metric, F.Cu at (138.5, 96.5)
- added U3: MCP3021, MCP3021:SOT-23, F.Cu at (144.0, 94.5)
- added U4: MCP3021, MCP3021:SOT-23, F.Cu at (144.0, 98.0)
- added U5: MCP23009-E_SS, MCP23009-E_SS:SOP65P780X200-20N, F.Cu at (140.6, 104.5)
- J1: value 24v DC -> ESC Left
- J10: value GND -> Switch 1; footprint Connector_Wire:SolderWire-0.75sqmm_1x01_D1.25mm_OD2.3mm -> Connector_JST:JST_XH_B4B-XH-AM_1x04_P2.50mm_Vertical
- J11: value GND -> Switch 2; footprint Connector_Wire:SolderWire-0.75sqmm_1x01_D1.25mm_OD2.3mm -> Connector_JST:JST_XH_B4B-XH-AM_1x04_P2.50mm_Vertical
- J2: value ESC Left -> ESC Right
- J3: value ESC Right -> 24v DC
- J5: value Strip light -> Panel; footprint Connector_JST:JST_XH_B2B-XH-A_1x02_P2.50mm_Vertical -> Connector_RJ:RJ45_Amphenol_RJHSE5380
- J6: value Joystick -> Strip light; footprint Connector_JST:JST_XH_B5B-XH-AM_1x05_P2.50mm_Vertical -> Connector_JST:JST_XH_B2B-XH-A_1x02_P2.50mm_Vertical
- J7: value Panel Lights -> Panel; footprint Connector_JST:JST_XH_B4B-XH-AM_1x04_P2.50mm_Vertical -> Connector_RJ:RJ45_Amphenol_RJHSE5380
- U1: value L7805 -> Pico; footprint Package_TO_SOT_SMD:TO-263-2 -> MCU_RaspberryPi_and_Boards:RPi_Pico_SMD_TH
- U2: value Pico -> L7805; footprint MCU_RaspberryPi_and_Boards:RPi_Pico_SMD_TH -> Package_TO_SOT_SMD:TO-263-2
- moved J6 60.8 mm to (60.0, 103.0), turned to 0 degrees
- moved Q2 50.7 mm to (152.0, 101.3)
- moved Q1 49.3 mm to (148.5, 101.3)
- moved H10 44.0 mm to (192.0, 56.0)
- moved G1 40.1 mm to (37.0, 123.0)
- moved J3 39.6 mm to (99.5, 74.2)
- moved T1 32.1 mm to (52.5, 94.5), turned to 0 degrees
- moved J2 30.9 mm to (53.0, 58.5)
- moved J7 27.9 mm to (124.8, 107.1)
- moved D1 23.9 mm to (92.0, 75.0)
- moved J10 19.1 mm to (148.9, 56.0), turned to 135 degrees
- moved J5 16.6 mm to (94.5, 87.8), turned to -90 degrees
- moved J1 15.8 mm to (53.0, 67.5)
- moved H8 15.5 mm to (122.0, 88.5)
- moved U2 13.5 mm to (97.0, 62.0), turned to 90 degrees
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Connections:
- J1 pad 1: +24V -> Net-(J1-Pad1)
- J3 pad 1: Net-(J3-Pad1) -> +24V
- J5 pad 1: Net-(J5-Pad1) -> +3V3
- J5 pad 2: +24V -> Net-(J5-Pad2)
- J6 pad 1: GND -> Net-(J6-Pad1)
- J6 pad 2: +3V3 -> +24V
- J7 pad 1: Net-(J7-Pad1) -> +3V3
- J7 pad 2: Net-(J7-Pad2) -> SCL
- J7 pad 3: Net-(J7-Pad3) -> SDA
- Q1 pad 3: Net-(J7-Pad3) -> Net-(J10-Pad3)
- Q1 pad 6: Net-(J7-Pad2) -> Net-(J11-Pad3)
- Q2 pad 3: Net-(J7-Pad1) -> Net-(J12-Pad3)
- T1 pad 2: Net-(J5-Pad1) -> Net-(J6-Pad1)
- T1 pad 3: GND -> Net-(J5-Pad5)
- U1 pad 1: +24V -> Net-(J1-Pad1)
- U1 pad 2: GND -> Net-(J2-Pad1)
- U1 pad 3: Net-(D1-Pad2) -> GND
- U2 pad 1: Net-(J2-Pad1) -> +24V
- U2 pad 2: Net-(J3-Pad1) -> GND
- U2 pad 3: GND -> Net-(D1-Pad2)
Routing:
- net Net-(J19-Pad1): track 109.1 -> 0.00 mm
- net Net-(J10-Pad2): track 0.00 -> 80.7 mm
- net Net-(J10-Pad3): track 0.00 -> 77.9 mm
- net Net-(J11-Pad2): track 0.00 -> 66.1 mm, vias 0 -> 1
- net Net-(J3-Pad1): track 58.1 -> 0.00 mm
- net Net-(J14-Pad1): track 51.9 -> 0.00 mm
- net Net-(J2-Pad1): track 50.7 -> 0.00 mm
- net Net-(J7-Pad6): track 0.00 -> 42.5 mm
- net Net-(J8-Pad1): track 41.0 -> 0.00 mm
- net Net-(D1-Pad1): track 40.1 -> 0.00 mm
- net Net-(J5-Pad1): track 39.8 -> 0.00 mm
- net Net-(J8-Pad2): track 39.0 -> 0.00 mm
- net Net-(J11-Pad3): track 0.00 -> 39.0 mm
- net Net-(J8-Pad4): track 48.7 -> 9.77 mm
- net SDA: track 0.00 -> 35.5 mm, vias 0 -> 3
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Other:
- board size 95 x 88.5 mm -> 107.5 x 86.9 mm

Commit message: Updated pcb and code
Parts:
- removed G2: LOGO, OneTouch_Logo:onetouchlogo
- removed H10, H12, H13, H4, H8, H9: MountingHole, MountingHole:MountingHole_3.2mm_M3
- removed H5, H6, H7: MountingHole, MountingHole:MountingHole_12.7mm
- removed J11: Switch 2, Connector_JST:JST_XH_B4B-XH-AM_1x04_P2.50mm_Vertical
- removed J12: Switch 3, Connector_JST:JST_XH_B4B-XH-AM_1x04_P2.50mm_Vertical
- removed J2: ESC Right, Connector_JST:JST_XH_B2B-XH-AM_1x02_P2.50mm_Vertical
- removed Q2: 2N7002HSX, Package_TO_SOT_SMD:SOT-363_SC-70-6
- removed T1: STD40NF10, STD40NF10:D_PAK
- added C1: 0.1µF, Capacitor_SMD:C_0603_1608Metric, F.Cu at (83.3, 96.6)
- added C2: 0.1µF, Capacitor_SMD:C_0603_1608Metric, F.Cu at (83.3, 86.4)
- added F1: SMD Fuse, Resistor_SMD:R_0603_1608Metric_Pad0.98x0.95mm_HandSolder, F.Cu at (93.5, 55.0)
- added J4: ESC Right, Connector_JST:JST_XH_B2B-XH-AM_1x02_P2.50mm_Vertical, F.Cu at (104.2, 69.5)
- added R3: 1K, Resistor_SMD:R_1206_3216Metric, F.Cu at (72.2, 85.8)
- added R4: 15K, Resistor_SMD:R_1206_3216Metric, F.Cu at (72.2, 88.0)
- H1, H2, H3: footprint MountingHole:MountingHole_3.2mm_M3 -> MountingHole:MountingHole_2.1mm
- J1: value ESC Left -> 24v; footprint Connector_JST:JST_XH_B2B-XH-AM_1x02_P2.50mm_Vertical -> Connector_Wire:SolderWire-1sqmm_1x02_P5.4mm_D1.4mm_OD2.7mm
- J10: value Switch 1 -> Switch 3; footprint Connector_JST:JST_XH_B4B-XH-AM_1x04_P2.50mm_Vertical -> Connector_Wire:SolderWire-0.1sqmm_1x04_P3.6mm_D0.4mm_OD1mm
- J3: value 24v DC -> ESC Left
- J5: value Panel -> OLED; footprint Connector_RJ:RJ45_Amphenol_RJHSE5380 -> Connector_Wire:SolderWire-0.1sqmm_1x04_P3.6mm_D0.4mm_OD1mm
- J6: value Strip light -> Joystick; footprint Connector_JST:JST_XH_B2B-XH-A_1x02_P2.50mm_Vertical -> Connector_Wire:SolderWire-0.1sqmm_1x05_P3.6mm_D0.4mm_OD1mm
- J7: value Panel -> Cutout; footprint Connector_RJ:RJ45_Amphenol_RJHSE5380 -> Connector_Wire:SolderWire-0.1sqmm_1x02_P3.6mm_D0.4mm_OD1mm
- J8: value Joystick -> Switch 1; footprint Connector_JST:JST_XH_B5B-XH-A_1x05_P2.50mm_Vertical -> Connector_Wire:SolderWire-0.1sqmm_1x04_P3.6mm_D0.4mm_OD1mm
- J9: value Cutout -> Switch 2; footprint Connector_JST:JST_XH_B2B-XH-AM_1x02_P2.50mm_Vertical -> Connector_Wire:SolderWire-0.1sqmm_1x04_P3.6mm_D0.4mm_OD1mm
- R1: value 1K -> 100k; footprint Resistor_SMD:R_1206_3216Metric -> Resistor_SMD:R_0603_1608Metric_Pad0.98x0.95mm_HandSolder
- R2: value 15K -> 18K; footprint Resistor_SMD:R_1206_3216Metric -> Resistor_SMD:R_0603_1608Metric_Pad0.98x0.95mm_HandSolder
- U3, U4: footprint MCP3021:SOT-23 -> Package_TO_SOT_SMD:SOT-23-5_HandSoldering
- moved J10 107.1 mm to (49.5, 96.0), turned to 0 degrees
- moved J8 101.3 mm to (49.5, 90.0), turned to 0 degrees
- moved Q1 85.3 mm to (64.0, 89.8)
- moved R2 80.8 mm to (69.5, 54.5), turned to 0 degrees
- moved R1 80.5 mm to (69.5, 57.5), turned to 180 degrees
- moved J7 77.9 mm to (49.5, 87.0), turned to 0 degrees
- moved G1 76.2 mm to (59.0, 50.0)
- moved J9 76.2 mm to (49.5, 93.0), turned to 0 degrees
- moved U5 69.3 mm to (72.2, 93.2)
- moved U4 61.4 mm to (83.3, 89.1), turned to 180 degrees
- moved U3 60.7 mm to (83.3, 93.9), turned to 180 degrees
- moved H2 52.5 mm to (105.0, 50.0)
- moved J6 49.1 mm to (107.0, 88.7), turned to 90 degrees
- moved H1 48.5 mm to (50.0, 50.0)
- moved J1 47.0 mm to (98.2, 55.0), turned to 90 degrees
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Connections:
- J1 pad 1: Net-(J1-Pad1) -> +BATT
- J3 pad 1: +24V -> Net-(J3-Pad1)
- J5 pad 1: +3V3 -> GND
- J5 pad 2: Net-(J5-Pad2) -> +3V3
- J5 pad 3: Net-(J5-Pad3) -> SCL
- J5 pad 4: +24V -> SDA
- J6 pad 1: Net-(J6-Pad1) -> GND
- J6 pad 2: +24V -> +3V3
- J7 pad 1: +3V3 -> GND
- J7 pad 2: SCL -> Net-(J7-Pad2)
- J8 pad 2: +3V3 -> Net-(J8-Pad2)
- J8 pad 4: Net-(J8-Pad4) -> +24V
- J9 pad 2: Net-(J7-Pad6) -> Net-(J9-Pad2)
- Q1 pad 3: Net-(J10-Pad3) -> Net-(J9-Pad3)
- Q1 pad 6: Net-(J11-Pad3) -> Net-(J8-Pad3)
- R1 pad 1: +3V3 -> +24V
- U1 pad 1: Net-(J1-Pad1) -> unconnected-(U1-Pad1)
- U1 pad 2: Net-(J2-Pad1) -> unconnected-(U1-Pad2)
- U1 pad 21: unconnected-(U1-Pad21) -> Net-(J4-Pad1)
- U1 pad 22: unconnected-(U1-Pad22) -> Net-(J3-Pad1)
- U1 pad 23: Net-(J5-Pad5) -> GND
- U1 pad 26: unconnected-(U1-Pad26) -> SDA
- U1 pad 27: Net-(T1-Pad1) -> SCL
- U1 pad 28: Net-(J5-Pad5) -> GND
- U1 pad 31: Net-(J5-Pad3) -> Net-(R1-Pad2)
- U1 pad 32: Net-(J5-Pad2) -> unconnected-(U1-Pad32)
- U1 pad 38: Net-(J5-Pad5) -> GND
- U1 pad 4: unconnected-(U1-Pad4) -> Net-(U1-Pad4)
- U3 pad 3: Net-(J8-Pad3) -> Net-(J6-Pad3)
- U4 pad 3: Net-(J8-Pad4) -> Net-(J6-Pad4)
- U5 pad 12: Net-(J12-Pad2) -> Net-(J10-Pad2)
- U5 pad 13: Net-(J11-Pad2) -> Net-(J9-Pad2)
- U5 pad 14: Net-(J10-Pad2) -> Net-(J8-Pad2)
- U5 pad 5: Net-(R1-Pad2) -> Net-(R3-Pad2)
- U5 pad 7: unconnected-(U5-Pad7) -> Net-(U1-Pad4)
- U5 pad 8: Net-(J8-Pad5) -> Net-(J6-Pad5)
- U5 pad 9: unconnected-(U5-Pad9) -> Net-(J7-Pad2)
Routing:
- net Net-(J10-Pad3): track 77.9 -> 0.00 mm
- net Net-(J6-Pad5): track 0.00 -> 67.2 mm, vias 0 -> 2
- net Net-(J11-Pad2): track 66.1 -> 0.00 mm, vias 1 -> 0
- net +3V3: track 61.0 -> 126.9 mm, vias 0 -> 2
- net Net-(J10-Pad2): track 80.7 -> 25.3 mm
- net Net-(J6-Pad3): track 0.00 -> 47.3 mm
- net Net-(Q1-Pad5): track 7.76 -> 54.9 mm
- net SCL: track 24.5 -> 70.5 mm, vias 3 -> 4
- net Net-(J8-Pad2): track 0.00 -> 42.9 mm
- net Net-(J7-Pad6): track 42.5 -> 0.00 mm
- net Net-(J11-Pad3): track 39.0 -> 0.00 mm
- net Net-(U1-Pad4): track 0.00 -> 37.8 mm, vias 0 -> 1
- net Net-(J9-Pad2): track 0.00 -> 36.1 mm
- net Net-(J6-Pad4): track 0.00 -> 34.0 mm
- net SDA: track 35.5 -> 69.2 mm, vias 3 -> 2
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Other:
- board size 107.5 x 86.9 mm -> 65 x 55 mm
- board text added: "Donie Kelly © 2023"
- board text removed: "Donie Kelly © 2022"

Commit message: Version 2.0 sent to manafacture
Other:
- board text added: "Donie Kelly © 2023 v2.0"
- board text removed: "Donie Kelly © 2023"
Changed lines of the file:
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@@
     (property "Sheetname" "")
     (attr exclude_from_pos_files)
-    (fp_text reference "J8" (at -2.1 0) (layer "F.SilkS")
+    (fp_text reference "J8" (at -2.25 0) (layer "F.SilkS")
       (effects (font (size 0.75 0.75) (thickness 0.15)))
     )
@@
     (property "Sheetname" "")
     (attr exclude_from_pos_files)
-    (fp_text reference "J9" (at -2 0) (layer "F.SilkS")
+    (fp_text reference "J9" (at -2.25 0) (layer "F.SilkS")
       (effects (font (size 0.75 0.75) (thickness 0.15)))
     )
@@
     (fp_line (start -1.6 -0.8) (end 1.6 -0.8) (layer "F.Fab") (width 0.1))
     (fp_line (start 1.6 -0.8) (end 1.6 0.8) (layer "F.Fab") (width 0.1))
-    (pad "1" smd roundrect (at -1.4625 0 180) (size 1.125 1.75) (layers "F.Cu" "F.Paste" "F.Mask") (roundrect_rratio 0.222222)
+    (pad "1" smd roundrect (at -1.4625 0 180) (size 1.125 1.75) (layers "F.Cu" "F.Paste" "F.Mask") (roundrect_rratio 0.2222222222)
       (net 51 "Net-(R3-Pad2)") (pintype "passive"))
-    (pad "2" smd roundrect (at 1.4625 0 180) (size 1.125 1.75) (layers "F.Cu" "F.Paste" "F.Mask") (roundrect_rratio 0.222222)
+    (pad "2" smd roundrect (at 1.4625 0 180) (size 1.125 1.75) (layers "F.Cu" "F.Paste" "F.Mask") (roundrect_rratio 0.2222222222)
       (net 2 "GND") (pintype "passive"))
     (model "${KICAD6_3DMODEL_DIR}/Resistor_SMD.3dshapes/R_1206_3216Metric.wrl"
@@
     (fp_line (start -2.45 -2.35) (end -2.45 3.4) (layer "F.Fab") (width 0.1))
     (pad "" np_thru_hole circle (at -1.6 2 90) (size 1.2 1.2) (drill 1.2) (layers *.Cu *.Mask))
-    (pad "1" thru_hole roundrect (at 0 0 90) (size 1.7 2) (drill 1) (layers *.Cu *.Mask) (roundrect_rratio 0.147059)
+    (pad "1" thru_hole roundrect (at 0 0 90) (size 1.7 2) (drill 1) (layers *.Cu *.Mask) (roundrect_rratio 0.1470588235)
       (net 58 "Net-(J4-Pad1)") (pinfunction "Pin_1") (pintype "passive"))
     (pad "2" thru_hole oval (at 2.5 0 90) (size 1.7 2) (drill 1) (layers *.Cu *.Mask)
@@
     (property "Sheetname" "")
     (attr exclude_from_pos_files)
-    (fp_text reference "J10" (at -2.5 0) (layer "F.SilkS")
+    (fp_text reference "J10" (at -2.75 0) (layer "F.SilkS")
       (effects (font (size 0.75 0.75) (thickness 0.15)))
     )
@@
     (property "Sheetname" "")
     (attr exclude_from_pos_files)
-    (fp_text reference "J1" (at 2.7 -2.58 90) (layer "F.SilkS")
+    (fp_text reference "J1" (at 2.7 -2.75 90) (layer "F.SilkS")
       (effects (font (size 1 1) (thickness 0.15)))
     )
@@
     (fp_circle (center 5.4 0) (end 6.75 0) (layer "F.Fab") (width 0.1) (fill none))
     (fp_circle (center 0 0) (end 1.35 0) (layer "F.Fab") (width 0.1) (fill none))
-    (pad "1" thru_hole roundrect (at 0 0 90) (size 2.75 2.75) (drill 1.75) (layers *.Cu *.Mask) (roundrect_rratio 0.090909)
+    (pad "1" thru_hole roundrect (at 0 0 90) (size 2.75 2.75) (drill 1.75) (layers *.Cu *.Mask) (roundrect_rratio 0.09090909091)
       (net 53 "+BATT") (pinfunction "Pin_1") (pintype "power_in"))
     (pad "2" thru_hole circle (at 5.4 0 90) (size 2.75 2.75) (drill 1.75) (layers *.Cu *.Mask)
@@
     (fp_line (start -1.6 -0.8) (end 1.6 -0.8) (layer "F.Fab") (width 0.1))
     (fp_line (start 1.6 -0.8) (end 1.6 0.8) (layer "F.Fab") (width 0.1))
-    (pad "1" smd roundrect (at -1.4625 0) (size 1.125 1.75) (layers "F.Cu" "F.Paste" "F.Mask") (roundrect_rratio 0.222222)
+    (pad "1" smd roundrect (at -1.4625 0) (size 1.125 1.75) (layers "F.Cu" "F.Paste" "F.Mask") (roundrect_rratio 0.2222222222)
       (net 8 "+3V3") (pintype "passive"))
-    (pad "2" smd roundrect (at 1.4625 0) (size 1.125 1.75) (layers "F.Cu" "F.Paste" "F.Mask") (roundrect_rratio 0.222222)
+    (pad "2" smd roundrect (at 1.4625 0) (size 1.125 1.75) (layers "F.Cu" "F.Paste" "F.Mask") (roundrect_rratio 0.2222222222)
       (net 51 "Net-(R3-Pad2)") (pintype "passive"))
     (model "${KICAD6_3DMODEL_DIR}/Resistor_SMD.3dshapes/R_1206_3216Metric.wrl"
@@
     (property "Sheetname" "")
     (attr exclude_from_pos_files)
-    (fp_text reference "J7" (at -2 0) (layer "F.SilkS")
+    (fp_text reference "J7" (at -2.25 0) (layer "F.SilkS")
       (effects (font (size 0.75 0.75) (thickness 0.15)))
     )
@@
     (fp_line (start 0 -1.35) (end 0.625 -2.35) (layer "F.Fab") (width 0.1))
     (pad "" np_thru_hole circle (at -1.6 2 90) (size 1.2 1.2) (drill 1.2) (layers *.Cu *.Mask))
-    (pad "1" thru_hole roundrect (at 0 0 90) (size 1.7 2) (drill 1) (layers *.Cu *.Mask) (roundrect_rratio 0.147059)
+    (pad "1" thru_hole roundrect (at 0 0 90) (size 1.7 2) (drill 1) (layers *.Cu *.Mask) (roundrect_rratio 0.1470588235)
       (net 57 "Net-(J3-Pad1)") (pinfunction "Pin_1") (pintype "passive"))
     (pad "2" thru_hole oval (at 2.5 0 90) (size 1.7 2) (drill 1) (layers *.Cu *.Mask)
@@
   (gr_arc (start 45 47.5) (mid 45.732233 45.732233) (end 47.5 45) (layer "Edge.Cuts") (width 0.1))
   (gr_line (start 47.5 45) (end 107.5 45) (layer "Edge.Cuts") (width 0.1))
-  (gr_text "Donie Kelly\n© 2023" (at 57 53.5) (layer "F.SilkS")
+  (gr_text "Donie Kelly\n© 2023 v2.0" (at 57 53.5) (layer "F.SilkS")
     (effects (font (size 0.7 0.7) (thickness 0.1)) (justify left))
   )

Commit message: library code update
Parts:
- J3: value ESC Left -> ESC 1 PCM
- J4: value ESC Right -> ESC 2 PCM
- Q1: value 2N7002HSX -> US6K1
Changed lines of the file:
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@@
       (effects (font (size 1 1) (thickness 0.15)))
     )
-    (fp_text value "ESC Right" (at 1.25 4.6 90) (layer "F.Fab")
+    (fp_text value "ESC 2 PCM" (at 1.25 4.6 90) (layer "F.Fab")
       (effects (font (size 1 1) (thickness 0.15)))
     )
@@
       (effects (font (size 0.75 0.75) (thickness 0.15)))
     )
-    (fp_text value "2N7002HSX" (at 0 2) (layer "F.Fab") hide
+    (fp_text value "US6K1" (at 0 2) (layer "F.Fab") hide
       (effects (font (size 1 1) (thickness 0.15)))
     )
@@
       (effects (font (size 1 1) (thickness 0.15)))
     )
-    (fp_text value "ESC Left" (at 1.25 4.6 90) (layer "F.Fab")
-      (effects (font (size 1 1) (thickness 0.15)))
-    )
+    (fp_text value "ESC 1 PCM" (at 1.25 4.6 90) (layer "F.Fab")
+      (effects (font (size 1 1) (thickness 0.15)))
+    )
