File: pcb/control/control.kicad_sch (KiCad schematic)
At the start: 15 parts, among them J1 24v DC, J2 ESC Left, J3 ESC Right, J4 Buttons, J5 Joystick, J6 Lights, Q1 2N7002HSX, Q2 2N7002HSX, U1 L7805, U2 Pico

Commit message: Updated pcb
Parts:
- added G1, G2: LOGO, OneTouch_Logo:onetouchlogo, symbol onetouchlogo:LOGO
- added H10, H11, H12, H13, H8, H9: MountingHole, MountingHole:MountingHole_3.2mm_M3, symbol Mechanical:MountingHole
- added H5, H6, H7: MountingHole, MountingHole:MountingHole_12.7mm, symbol Mechanical:MountingHole
- added J10, J11, J13: GND, Connector_Wire:SolderWire-0.75sqmm_1x01_D1.25mm_OD2.3mm, symbol Connector_Generic:Conn_01x01
- added J12, J9: Conn_01x04_Female, symbol Connector:Conn_01x04_Female
- added J14: 1, Connector_Wire:SolderWire-0.75sqmm_1x01_D1.25mm_OD2.3mm, symbol Connector_Generic:Conn_01x01
- added J15: 2, Connector_Wire:SolderWire-0.75sqmm_1x01_D1.25mm_OD2.3mm, symbol Connector_Generic:Conn_01x01
- added J16: 3, Connector_Wire:SolderWire-0.75sqmm_1x01_D1.25mm_OD2.3mm, symbol Connector_Generic:Conn_01x01
- added J17, J18, J19: LED +, Connector_Wire:SolderWire-0.75sqmm_1x01_D1.25mm_OD2.3mm, symbol Connector_Generic:Conn_01x01
- added J20, J21, J22: LED -, Connector_Wire:SolderWire-0.75sqmm_1x01_D1.25mm_OD2.3mm, symbol Connector_Generic:Conn_01x01
- added J23: Joystick, Connector_Wire:SolderWire-0.75sqmm_1x05_P7mm_D1.25mm_OD3.5mm, symbol Connector_Generic:Conn_01x05
- added J24: Joystick, Connector_JST:JST_XH_B5B-XH-AM_1x05_P2.50mm_Vertical, symbol Connector:Conn_01x05_Male
- added J25: Panel Lights, Connector_JST:JST_XH_B4B-XH-AM_1x04_P2.50mm_Vertical, symbol Connector:Conn_01x04_Male
- added J26: Panel Buttons, Connector_JST:JST_XH_B4B-XH-AM_1x04_P2.50mm_Vertical, symbol Connector:Conn_01x04_Male
- added J5: Strip light, Connector_JST:JST_XH_B2B-XH-A_1x02_P2.50mm_Vertical, symbol Connector:Conn_01x02_Male
- added J8: Joystick, symbol Connector:Conn_01x05_Female
- added T1: STD40NF10, STD40NF10:D_PAK, symbol STD40NF10:STD40NF10
- J4: value Buttons -> Panel Buttons
- J7: renamed from J6; value Lights -> Panel Lights
- renumbered J5 to J6
Connections:
- net +24V: now also J5.2 (Pin_2)
- net GND: now also J10.1 (Pin_1), J11.1 (Pin_1), J13.1 (Pin_1), J23.1 (Pin_1), J24.1 (Pin_1), J26.4 (Pin_4), J8.5 (Pin_5), J9.4 (Pin_4), T1.3 (S)
- net at U2.20 (GPIO15): now also T1.1 (G)
- net +3V3: now reaches J6.2 (Pin_2), U2.36 (3V3)
- new net: J16.1 (Pin_1), J26.1 (Pin_1), J9.1 (Pin_1)
- new net: J12.1 (Pin_1), J22.1 (Pin_1), J25.1 (Pin_1)
- new net: J12.4 (Pin_4), J17.1 (Pin_1), J18.1 (Pin_1), J19.1 (Pin_1), J25.4 (Pin_4)
- new net: J15.1 (Pin_1), J26.2 (Pin_2), J9.2 (Pin_2)
- new net: J14.1 (Pin_1), J26.3 (Pin_3), J9.3 (Pin_3)
- new net: J12.3 (Pin_3), J20.1 (Pin_1), J25.3 (Pin_3)
- new net: J12.2 (Pin_2), J21.1 (Pin_1), J25.2 (Pin_2)
- new net: J23.2 (Pin_2), J24.2 (Pin_2), J8.4 (Pin_4)
- new net: J23.3 (Pin_3), J24.3 (Pin_3), J8.3 (Pin_3)
- new net: J23.4 (Pin_4), J24.4 (Pin_4), J8.2 (Pin_2)
- new net: J23.5 (Pin_5), J24.5 (Pin_5), J8.1 (Pin_1)
- new net: J5.1 (Pin_1), T1.2 (D)
- no-connect marks 3 -> 22

Commit message: v2 of design
Parts:
- removed H11: MountingHole, MountingHole:MountingHole_3.2mm_M3, symbol Mechanical:MountingHole
- removed J10, J11, J13: GND, Connector_Wire:SolderWire-0.75sqmm_1x01_D1.25mm_OD2.3mm, symbol Connector_Generic:Conn_01x01
- removed J12, J9: Conn_01x04_Female, symbol Connector:Conn_01x04_Female
- removed J14: 1, Connector_Wire:SolderWire-0.75sqmm_1x01_D1.25mm_OD2.3mm, symbol Connector_Generic:Conn_01x01
- removed J15: 2, Connector_Wire:SolderWire-0.75sqmm_1x01_D1.25mm_OD2.3mm, symbol Connector_Generic:Conn_01x01
- removed J16: 3, Connector_Wire:SolderWire-0.75sqmm_1x01_D1.25mm_OD2.3mm, symbol Connector_Generic:Conn_01x01
- removed J17, J18, J19: LED +, Connector_Wire:SolderWire-0.75sqmm_1x01_D1.25mm_OD2.3mm, symbol Connector_Generic:Conn_01x01
- removed J20, J21, J22: LED -, Connector_Wire:SolderWire-0.75sqmm_1x01_D1.25mm_OD2.3mm, symbol Connector_Generic:Conn_01x01
- removed J24, J6: Joystick, Connector_JST:JST_XH_B5B-XH-AM_1x05_P2.50mm_Vertical, symbol Connector:Conn_01x05_Male
- removed J25, J7: Panel Lights, Connector_JST:JST_XH_B4B-XH-AM_1x04_P2.50mm_Vertical, symbol Connector:Conn_01x04_Male
- removed J26, J4: Panel Buttons, Connector_JST:JST_XH_B4B-XH-AM_1x04_P2.50mm_Vertical, symbol Connector:Conn_01x04_Male
- removed J8: Joystick, symbol Connector:Conn_01x05_Female
- added J10: Switch 1, Connector_JST:JST_XH_B4B-XH-AM_1x04_P2.50mm_Vertical, symbol Connector:Conn_01x04_Male
- added J11: Switch 2, Connector_JST:JST_XH_B4B-XH-AM_1x04_P2.50mm_Vertical, symbol Connector:Conn_01x04_Male
- added J12: Switch 3, Connector_JST:JST_XH_B4B-XH-AM_1x04_P2.50mm_Vertical, symbol Connector:Conn_01x04_Male
- added J4: Conn_01x02_Male, symbol Connector:Conn_01x02_Male
- added J5, J7: Panel, Connector_RJ:RJ45_Amphenol_RJHSE5380, symbol Connector:RJ45_Shielded
- added J9: Cutout, Connector_JST:JST_XH_B2B-XH-AM_1x02_P2.50mm_Vertical, symbol Connector:Conn_01x02_Male
- added K1: ADW11, Relay_THT:Relay_1P1T_NO_10x24x18.8mm_Panasonic_ADW11xxxxW_THT, symbol Relay:ADW11
- added R1: 1K, Resistor_SMD:R_1206_3216Metric, symbol Device:R
- added R2: 15K, Resistor_SMD:R_1206_3216Metric, symbol Device:R
- added U3, U4: MCP3021, SOT-23, symbol MCP3021:MCP3021
- added U5: MCP23009-E_SS, SOP65P780X200-20N, symbol MCP23009-E_SS:MCP23009-E_SS
- J3: renamed from J1; symbol Connector:Conn_01x02_Male -> Connector:Conn_01x02_Female
- J8: renamed from J23; footprint Connector_Wire:SolderWire-0.75sqmm_1x05_P7mm_D1.25mm_OD3.5mm -> Connector_JST:JST_XH_B5B-XH-A_1x05_P2.50mm_Vertical; symbol Connector_Generic:Conn_01x05 -> Connector:Conn_01x05_Male
- T1: footprint STD40NF10:D_PAK -> D_PAK
- renumbered J2 to J1, J3 to J2, J5 to J6, U2 to U1, U1 to U2
Connections:
- net +24V: now also J10.4 (Pin_4), J11.4 (Pin_4), J12.4 (Pin_4), J5.4, J7.4
- net +3V3: now also J8.2 (Pin_2), J5.1, J7.1, R1.1, U3.1 (VCC), U4.1 (VCC), U5.1 (VDD), U5.6 (~{RESET})
- net GND: now also J10.1 (Pin_1), J11.1 (Pin_1), J12.1 (Pin_1), J4.2 (Pin_2), J5.SH, J7.5, J7.7, J7.8, J7.SH, J9.1 (Pin_1), R2.2, U3.2 (GND), U4.2 (GND), U5.20 (VSS); no longer T1.3 (S), U1.23 (GND), U1.28 (GND), U1.38 (GND)
- net at Q2.3 (D): now also J12.3 (Pin_3)
- net at Q1.6 (D): now also J11.3 (Pin_3)
- net at Q1.3 (D): now also J10.3 (Pin_3)
- net at U1.20 (GPIO15): no longer T1.1 (G)
- net at U1.26 (GPIO20): no longer Q2.2 (G)
- net at U1.27 (GPIO21): now also T1.1 (G); no longer Q1.5 (G)
- net at U1.29 (GPIO22): no longer Q1.2 (G)
- net at U1.31 (GPIO26_ADC0): now also J5.3
- net at U1.32 (GPIO27_ADC1): now also J5.2
- net at J8.3 (Pin_3): now also U3.3 (AIN)
- net at J8.4 (Pin_4): now also U4.3 (AIN)
- net at J8.5 (Pin_5): now also U5.8 (GP0)
- new net: J10.2 (Pin_2), U5.14 (GP4)
- new net: J5.5, J5.7, J5.8, T1.3 (S), U1.23 (GND), U1.28 (GND), U1.38 (GND)
- new net: R1.2, R2.1, U5.5 (ADDR)
- new net: J12.2 (Pin_2), U5.12 (GP2)
- new net: J4.1 (Pin_1), K1.3
- new net: Q2.2 (G), U5.15 (GP5)
- new net: Q1.2 (G), U5.17 (GP7)
- new net: Q1.5 (G), U5.16 (GP6)
- new net: J7.6, J9.2 (Pin_2)
- new net: J11.2 (Pin_2), U5.13 (GP3)
- new net SCL: J7.2, U3.5 (SCL), U4.5 (SCL), U5.3 (SCL)
- new net SDA: J7.3, U3.4 (SDA), U4.4 (SDA), U5.4 (SDA)
- no-connect marks 22 -> 40
Other:
- moved on the sheet: H1, H10, H12, H13, H2, H3, H4, H5, H6, H7, H8, H9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

Commit message: Updated pcb and code
Parts:
- removed G2: LOGO, OneTouch_Logo:onetouchlogo, symbol onetouchlogo:LOGO
- removed H10, H12, H13, H4, H8, H9: MountingHole, MountingHole:MountingHole_3.2mm_M3, symbol Mechanical:MountingHole
- removed H5, H6, H7: MountingHole, MountingHole:MountingHole_12.7mm, symbol Mechanical:MountingHole
- removed J5, J7: Panel, Connector_RJ:RJ45_Amphenol_RJHSE5380, symbol Connector:RJ45_Shielded
- removed J6: Strip light, Connector_JST:JST_XH_B2B-XH-A_1x02_P2.50mm_Vertical, symbol Connector:Conn_01x02_Male
- removed T1: STD40NF10, D_PAK, symbol STD40NF10:STD40NF10
- added BT1: Battery 21v, symbol Device:Battery
- added C1, C2: 0.1µF, Capacitor_SMD:C_0603_1608Metric, symbol Device:C
- added F1: SMD Fuse, Resistor_SMD:R_0603_1608Metric_Pad0.98x0.95mm_HandSolder, symbol Device:Fuse
- added F2: 100A, Resistor_SMD:R_0603_1608Metric_Pad0.98x0.95mm_HandSolder, symbol Device:Fuse
- added J5: OLED, Connector_Wire:SolderWire-0.1sqmm_1x04_P3.6mm_D0.4mm_OD1mm, symbol Connector:Conn_01x04_Male
- added M1: ESC1, symbol Motor:Motor_DC
- added M2: ESC2, symbol Motor:Motor_DC
- added unit 2 of Q2
- added R1: 100k, Resistor_SMD:R_0603_1608Metric_Pad0.98x0.95mm_HandSolder, symbol Device:R
- added R2: 18K, Resistor_SMD:R_0603_1608Metric_Pad0.98x0.95mm_HandSolder, symbol Device:R
- added SW1: Master SW, symbol Switch:SW_SPST
- H1, H2, H3: footprint MountingHole:MountingHole_3.2mm_M3 -> MountingHole:MountingHole_2.1mm
- J1: renamed from J3; value 24v DC -> 24v; footprint Connector_JST:JST_XH_B2B-XH-AM_1x02_P2.50mm_Vertical -> Connector_Wire:SolderWire-1sqmm_1x02_P5.4mm_D1.4mm_OD2.7mm
- J10: renamed from J12; footprint Connector_JST:JST_XH_B4B-XH-AM_1x04_P2.50mm_Vertical -> Connector_Wire:SolderWire-0.1sqmm_1x04_P3.6mm_D0.4mm_OD1mm
- J6: renamed from J8; footprint Connector_JST:JST_XH_B5B-XH-A_1x05_P2.50mm_Vertical -> Connector_Wire:SolderWire-0.1sqmm_1x05_P3.6mm_D0.4mm_OD1mm
- J7: renamed from J9; footprint Connector_JST:JST_XH_B2B-XH-AM_1x02_P2.50mm_Vertical -> Connector_Wire:SolderWire-0.1sqmm_1x02_P3.6mm_D0.4mm_OD1mm
- J8: renamed from J10; footprint Connector_JST:JST_XH_B4B-XH-AM_1x04_P2.50mm_Vertical -> Connector_Wire:SolderWire-0.1sqmm_1x04_P3.6mm_D0.4mm_OD1mm
- J9: renamed from J11; footprint Connector_JST:JST_XH_B4B-XH-AM_1x04_P2.50mm_Vertical -> Connector_Wire:SolderWire-0.1sqmm_1x04_P3.6mm_D0.4mm_OD1mm
- U3, U4: footprint SOT-23 -> Package_TO_SOT_SMD:SOT-23-5_HandSoldering
- U5: footprint SOP65P780X200-20N -> MCP23009-E_SS:SOP65P780X200-20N
- renumbered J4 to J2, J1 to J3, J2 to J4, R1 to R3, R2 to R4
Connections:
- net +24V: now also F1.2, R1.1; no longer J1.1 (Pin_1)
- net +3V3: now also C1.1, C2.1, J5.2 (Pin_2)
- net GND: now also K1.1, U1.23 (GND), U1.28 (GND), U1.38 (GND), BT1.2 (-), C1.2, C2.2, J5.1 (Pin_1), M1.2 (-), M2.2 (-), R2.2
- net SCL: now also U1.27 (GPIO21), J5.3 (Pin_3)
- net SDA: now also U1.26 (GPIO20), J5.4 (Pin_4)
- net at J8.3 (Pin_3): now also Q1.6 (D); no longer Q1.3 (D)
- net at U1.1 (GPIO0): no longer J3.1 (Pin_1)
- net at U1.2 (GPIO1): no longer J4.1 (Pin_1)
- net at U1.21 (GPIO16): now also J4.1 (Pin_1)
- net at U1.22 (GPIO17): now also J3.1 (Pin_1)
- net at U1.31 (GPIO26_ADC0): now also R1.2, R2.1
- net at U1.4 (GPIO2): now also U5.7 (INT)
- net at J10.3 (Pin_3): now also Q2.6 (D); no longer Q2.3 (D)
- net at J9.3 (Pin_3): now also Q1.3 (D); no longer Q1.6 (D)
- net at K1.5: now also F2.1, M1.1 (+), M2.1 (+), SW1.2 (B)
- net at K1.6: now also SW1.1 (A)
- net at J7.2 (Pin_2): now also U5.9 (GP1)
- new net: BT1.1 (+), F2.2
- new net +BATT: F1.1, J1.1 (Pin_1)
- no-connect marks 40 -> 36
Other:
- moved on the sheet: D1, H1, H2, H3, J10, J2, J3, J4, J6, J7, J8, J9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

Commit message: Updated code
Parts:
- J3: value ESC Left -> ESC 1 PCM
- J4: value ESC Right -> ESC 2 PCM
- Q1, Q2: value 2N7002HSX -> US6K1
Changed lines of the file:
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@@
       (effects (font (size 1.27 1.27)) (justify right))
     )
-    (property "Value" "ESC Right" (id 1) (at 95.9612 164.2622 0)
+    (property "Value" "ESC 2 PCM" (id 1) (at 95.9612 164.2622 0)
       (effects (font (size 1.27 1.27)) (justify right))
     )
@@
       (effects (font (size 1.27 1.27)) (justify left))
     )
-    (property "Value" "2N7002HSX" (id 1) (at 243.967 131.2422 0)
+    (property "Value" "US6K1" (id 1) (at 243.967 131.2422 0)
       (effects (font (size 1.27 1.27)) (justify left))
     )
@@
       (effects (font (size 1.27 1.27) italic) (justify left) hide)
     )
-    (property "Datasheet" "https://www.farnell.com/datasheets/3669737.pdf" (id 3) (at 243.84 137.16 0)
+    (property "Datasheet" "https://4donline.ihs.com/images/VipMasterIC/IC/ROHM/ROHM-S-A0008995927/ROHM-S-A0008995927-1.pdf?hkey=6D3A4C79FDBF58556ACFDE234799DDF0" (id 3) (at 243.84 137.16 0)
       (effects (font (size 1.27 1.27)) (justify left) hide)
     )
@@
       (effects (font (size 1.27 1.27)) (justify left))
     )
-    (property "Value" "2N7002HSX" (id 1) (at 238.887 103.3022 0)
+    (property "Value" "US6K1" (id 1) (at 238.887 103.3022 0)
       (effects (font (size 1.27 1.27)) (justify left))
     )
@@
       (effects (font (size 1.27 1.27) italic) (justify left) hide)
     )
-    (property "Datasheet" "https://www.farnell.com/datasheets/3669737.pdf" (id 3) (at 238.76 109.22 0)
+    (property "Datasheet" "https://4donline.ihs.com/images/VipMasterIC/IC/ROHM/ROHM-S-A0008995927/ROHM-S-A0008995927-1.pdf?hkey=6D3A4C79FDBF58556ACFDE234799DDF0" (id 3) (at 238.76 109.22 0)
       (effects (font (size 1.27 1.27)) (justify left) hide)
     )
@@
       (effects (font (size 1.27 1.27)) (justify left))
     )
-    (property "Value" "2N7002HSX" (id 1) (at 243.967 152.8322 0)
+    (property "Value" "US6K1" (id 1) (at 243.967 152.8322 0)
       (effects (font (size 1.27 1.27)) (justify left))
     )
@@
       (effects (font (size 1.27 1.27) italic) (justify left) hide)
     )
-    (property "Datasheet" "https://www.farnell.com/datasheets/3669737.pdf" (id 3) (at 243.84 158.75 0)
+    (property "Datasheet" "https://4donline.ihs.com/images/VipMasterIC/IC/ROHM/ROHM-S-A0008995927/ROHM-S-A0008995927-1.pdf?hkey=6D3A4C79FDBF58556ACFDE234799DDF0" (id 3) (at 243.84 158.75 0)
       (effects (font (size 1.27 1.27)) (justify left) hide)
     )
@@
       (effects (font (size 1.27 1.27)) (justify left))
     )
-    (property "Value" "2N7002HSX" (id 1) (at 241.427 117.2722 0)
+    (property "Value" "US6K1" (id 1) (at 241.427 117.2722 0)
       (effects (font (size 1.27 1.27)) (justify left))
     )
@@
       (effects (font (size 1.27 1.27) italic) (justify left) hide)
     )
-    (property "Datasheet" "https://www.farnell.com/datasheets/3669737.pdf" (id 3) (at 241.3 123.19 0)
+    (property "Datasheet" "https://4donline.ihs.com/images/VipMasterIC/IC/ROHM/ROHM-S-A0008995927/ROHM-S-A0008995927-1.pdf?hkey=6D3A4C79FDBF58556ACFDE234799DDF0" (id 3) (at 241.3 123.19 0)
       (effects (font (size 1.27 1.27)) (justify left) hide)
     )
@@
       (effects (font (size 1.27 1.27)) (justify right))
     )
-    (property "Value" "ESC Left" (id 1) (at 95.9612 157.9122 0)
+    (property "Value" "ESC 1 PCM" (id 1) (at 95.9612 157.9122 0)
       (effects (font (size 1.27 1.27)) (justify right))
     )
@@
     )
     (path "/8a19e74a-359a-44af-90e8-1e0d716771fe"
-      (reference "J3") (unit 1) (value "ESC Left") (footprint "Connector_JST:JST_XH_B2B-XH-AM_1x02_P2.50mm_Vertical")
+      (reference "J3") (unit 1) (value "ESC 1 PCM") (footprint "Connector_JST:JST_XH_B2B-XH-AM_1x02_P2.50mm_Vertical")
     )
     (path "/443a5989-0cb2-4225-83d8-4313f11b01a7"
-      (reference "J4") (unit 1) (value "ESC Right") (footprint "Connector_JST:JST_XH_B2B-XH-AM_1x02_P2.50mm_Vertical")
+      (reference "J4") (unit 1) (value "ESC 2 PCM") (footprint "Connector_JST:JST_XH_B2B-XH-AM_1x02_P2.50mm_Vertical")
     )
     (path "/fb965fb4-a702-4b6d-8417-7eb0f04bfe62"
@@
     )
     (path "/84837aa9-7140-4fac-be22-3a17767cde79"
-      (reference "Q1") (unit 1) (value "2N7002HSX") (footprint "Package_TO_SOT_SMD:SOT-363_SC-70-6")
+      (reference "Q1") (unit 1) (value "US6K1") (footprint "Package_TO_SOT_SMD:SOT-363_SC-70-6")
     )
     (path "/898d718d-81cb-4e75-aca2-e4f27e81d43d"
-      (reference "Q1") (unit 2) (value "2N7002HSX") (footprint "Package_TO_SOT_SMD:SOT-363_SC-70-6")
+      (reference "Q1") (unit 2) (value "US6K1") (footprint "Package_TO_SOT_SMD:SOT-363_SC-70-6")
     )
     (path "/7e526690-9753-4464-9bb8-5720c89f8bc6"
-      (reference "Q2") (unit 1) (value "2N7002HSX") (footprint "Package_TO_SOT_SMD:SOT-363_SC-70-6")
+      (reference "Q2") (unit 1) (value "US6K1") (footprint "Package_TO_SOT_SMD:SOT-363_SC-70-6")
     )
     (path "/88ba96a2-3795-491d-8335-be7d86097f53"
-      (reference "Q2") (unit 2) (value "2N7002HSX") (footprint "Package_TO_SOT_SMD:SOT-363_SC-70-6")
+      (reference "Q2") (unit 2) (value "US6K1") (footprint "Package_TO_SOT_SMD:SOT-363_SC-70-6")
     )
     (path "/42124afc-687e-44b5-a9e7-3d74e0a7e27c"
